File: ADC/Cartpole_ADC_interface.kicad_pcb (KiCad board)
At the start: 2 copper layers, 24 x 18.5 mm, 10 parts, among them J1 Socket for JST XH, J2 Socket for potentiometer leads

Commit message: Fit left size of ADC interface board to the PMOD spec
Parts:
- C1: value 20 -> 20 uf
- C2: value 4.7 -> 4.7 uf
- C3: value 1 -> 1 uf
- FB1: value FerriteBead -> Ferrite Bead
- R1: value 12000 -> 12K
- R2: value 100 -> 100R
Other:
- board size 24 x 18.5 mm -> 25.8 x 18.5 mm
Changed lines of the file:
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@@
 			)
 		)
-		(property "Value" "1"
+		(property "Value" "1 uf"
 			(at 0 1.85 0)
 			(layer "F.Fab")
@@
 			)
 		)
-		(property "Value" "4.7"
+		(property "Value" "4.7 uf"
 			(at 0 1.85 90)
 			(layer "F.Fab")
@@
 			)
 		)
-		(property "Value" "100"
+		(property "Value" "100R"
 			(at 0 1.82 0)
 			(layer "F.Fab")
@@
 			)
 		)
-		(property "Value" "20"
+		(property "Value" "20 uf"
 			(at 0 1.85 0)
 			(layer "F.Fab")
@@
 			)
 		)
-		(property "Value" "FerriteBead"
+		(property "Value" "Ferrite Bead"
 			(at 0 1.85 0)
 			(layer "F.Fab")
@@
 			)
 		)
-		(property "Value" "12000"
+		(property "Value" "12K"
 			(at 0 1.82 90)
 			(layer "F.Fab")
@@
 	)
 	(gr_rect
-		(start 88.5 87)
+		(start 86.75 87)
 		(end 112.5 105.5)
 		(stroke

Commit message: Grounded pin 9 of the adc interface board (apparently this is atually necessary)
Connections:
- JA1 pad 9: unconnected-(JA1-Pin_9-Pad9) -> GND
Routing:
- net GND: track 25.2 -> 31.3 mm
Changed lines of the file:
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@@
 	(net 10 "unconnected-(JA1-Pin_1-Pad1)")
 	(net 11 "unconnected-(JA1-Pin_10-Pad10)")
-	(net 12 "unconnected-(JA1-Pin_9-Pad9)")
-	(net 13 "unconnected-(JA1-Pin_11-Pad11)")
-	(net 14 "unconnected-(JA1-Pin_8-Pad8)")
-	(net 15 "unconnected-(JA1-Pin_4-Pad4)")
+	(net 12 "unconnected-(JA1-Pin_11-Pad11)")
+	(net 13 "unconnected-(JA1-Pin_8-Pad8)")
+	(net 14 "unconnected-(JA1-Pin_4-Pad4)")
 	(footprint "Connector_PinHeader_2.54mm:PinHeader_1x03_P2.54mm_Vertical"
 		(layer "F.Cu")
@@
 			(layers "*.Cu" "*.Mask" "F.SilkS")
 			(remove_unused_layers no)
-			(net 15 "unconnected-(JA1-Pin_4-Pad4)")
+			(net 14 "unconnected-(JA1-Pin_4-Pad4)")
 			(pinfunction "Pin_4")
 			(pintype "passive")
@@
 			(layers "*.Cu" "*.Mask" "F.SilkS")
 			(remove_unused_layers no)
-			(net 14 "unconnected-(JA1-Pin_8-Pad8)")
+			(net 13 "unconnected-(JA1-Pin_8-Pad8)")
 			(pinfunction "Pin_8")
 			(pintype "passive")
@@
 			(layers "*.Cu" "*.Mask" "F.SilkS")
 			(remove_unused_layers no)
-			(net 12 "unconnected-(JA1-Pin_9-Pad9)")
+			(net 2 "GND")
 			(pinfunction "Pin_9")
 			(pintype "passive")
@@
 			(layers "*.Cu" "*.Mask" "F.SilkS")
 			(remove_unused_layers no)
-			(net 13 "unconnected-(JA1-Pin_11-Pad11)")
+			(net 12 "unconnected-(JA1-Pin_11-Pad11)")
 			(pinfunction "Pin_11")
 			(pintype "passive")
@@
 	)
 	(segment
+		(start 93.04 100.08)
+		(end 91.75 98.79)
+		(width 0.2)
+		(layer "F.Cu")
+		(net 2)
+	)
+	(segment
 		(start 100.125 96.5)
 		(end 100 96.5)
@@
 	)
 	(segment
+		(start 91.75 98.79)
+		(end 91.75 96.25)
+		(width 0.2)
+		(layer "F.Cu")
+		(net 2)
+	)
+	(segment
 		(start 98.5 91.5)
 		(end 98.5 94.875)
@@
 		(width 0.2)
 		(layer "F.Cu")
+		(net 2)
+	)
+	(segment
+		(start 91.75 96.25)
+		(end 90.5 95)
+		(width 0.2)
+		(layer "F.Cu")
